File: src/ELIESTER_V2/16BIT_ADC_ADS1115.kicad_sch (KiCad schematic)
At the start: 3 parts

Commit message: update on antenna an LAN side
Parts:
- U?: footprint Package_SO:TSSOP-10_3x3mm_P0.5mm -> Package_SO:VSSOP-10_3x3mm_P0.5mm
Changed lines of the file:
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@@
       (effects (font (size 1.27 1.27)) (justify right))
     )
-    (property "Footprint" "Package_SO:TSSOP-10_3x3mm_P0.5mm" (at 130.175 92.075 0)
+    (property "Footprint" "Package_SO:VSSOP-10_3x3mm_P0.5mm" (at 130.175 92.075 0)
       (effects (font (size 1.27 1.27)) hide)
     )
