File: src/ELIESTER_V2/ELIESTER_V2.kicad_pcb (KiCad board)
At the start: 4 copper layers, 102 x 86.2 mm, 309 parts, among them J1 Barrel_Jack_Switch, J10 Conn_01x04, J11 SIM_Card, J2 SCREEN CONN FPC 10PIN 1MM, J3 Conn_01x04, J4 Conn_01x04, J5 USB_B_Micro, J6 Conn_01x04, J7 Conn_01x04, J8 RJ45_Bel_SI-60062-F, J9 Conn_01x04, Q1 MMBT3904, Q11 MMBT3904, Q12 MMBT3904, Q2 MMBT3904, Q3 DMP3056L-7, Q4 DMP3056L-7, Q5 SI2302-HXY, Q6 DMP3056L-7, Q7 BSN20, Q8 BSN20, SW1 SW_Push, SW2 SW_Push, SW3 SW_Push, U1 WAS3157B, U10 PC817, U11 PC817, U12 W5500, U13 TBU-CA065-200-WH, U14 TPS56339DDC, U15 MAX485E, U16 TBU-CA065-200-WH, U17 SN74AHC1G125, U18 PC817, U19 ADS1115IDGS, U2 MAX3232, U20 PC817, U21 PC817, U22 PC817, U23 PC817, U24 PCF8574A, U25 SY8089AAAC, U26 SIM7000G, U3 ESP32 Wroom, U4 CH340T(SSOP20W), U5 WAS3157B, U6 PC817, U7 PC817, U8 TPS54331, U9 DS3231MZ_V__NRND, Y1 12MHz, Y2 25MHz

Commit message: schematic update and gerber updates with corrections
Parts:
- removed Q11, Q12: MMBT3904, Package_TO_SOT_SMD:SOT-23
- removed R77: 100K, Resistor_SMD:R_0603_1608Metric
- removed R78: 4.7K, Resistor_SMD:R_0603_1608Metric
- added F1: JK30-250, greencharge-footprints:fuse-JK30-200, F.Cu at (176.2, 88.9)
- added F2: JK30-250, Fuse:Fuse_1210_3225Metric_Pad1.42x2.65mm_HandSolder, F.Cu at (169.9, 106.8)
- added Q10: 2N7002, Package_TO_SOT_SMD:SOT-23, B.Cu at (198.4, 117.8)
- added Q9: 2N7002, Package_TO_SOT_SMD:SOT-23, B.Cu at (199.3, 122.8)
- added R67: 10K, Resistor_SMD:R_0402_1005Metric, B.Cu at (196.8, 122.8)
- added R68: 10K, Resistor_SMD:R_0402_1005Metric, B.Cu at (200.4, 120.6)
- added R69: 1K, Resistor_SMD:R_0402_1005Metric, B.Cu at (197.8, 120.6)
- C57, C58: value 22p -> 16p
- R1: value 2K -> 10R
- R74: value 4.7K -> 10K; footprint Resistor_SMD:R_0603_1608Metric -> Resistor_SMD:R_0402_1005Metric
- R75: value 100K -> 10K; footprint Resistor_SMD:R_0603_1608Metric -> Resistor_SMD:R_0402_1005Metric
- R76: value 4.7K -> 1K; footprint Resistor_SMD:R_0603_1608Metric -> Resistor_SMD:R_0402_1005Metric
- moved R75 8.10 mm to (199.9, 115.5)
- moved C23 6.70 mm to (174.1, 105.6)
- moved C24 5.54 mm to (174.2, 106.7)
- moved L3 5.00 mm to (172.9, 103.8), turned to 0 degrees
- moved R1 4.87 mm to (179.0, 98.8), turned to 90 degrees
- moved R74 4.04 mm to (195.9, 117.1)
- moved Z1 3.80 mm to (179.3, 94.1)
- moved R76 2.50 mm to (197.8, 115.5)
- moved C25 1.20 mm to (169.1, 104.6)
- moved C12 1.15 mm to (169.2, 103.5)
Connections:
- C23 pad 1: Net-(J5-VBUS) -> Net-(C23-Pad1)
- C24 pad 1: Net-(J5-VBUS) -> Net-(C23-Pad1)
- J1 pad 1: +24V -> Net-(F1-Pad1)
- L3 pad 2: Net-(J5-VBUS) -> Net-(C23-Pad1)
- R49 pad 2: /SPI_ETH_INTERFACE_W5500/3V3A -> /SPI_ETH_INTERFACE_W5500/3V3D
- R74 pad 1: Net-(Q11-B) -> VDD_EXT
- R74 pad 2: VDD_EXT -> Net-(Q10-S)
- R75 pad 1: /ESP32_MCU/soft_uart_rx -> +3V3
- R75 pad 2: +3V3 -> /ESP32_MCU/soft_uart_tx
- R76 pad 1: Net-(Q12-B) -> /GSM_GPRS_MODULE_SIM7000G/MOSFET_LOGIC_LEVEL_TRANSLATOR/LOW_SIDE_LOGIC_SIGNAL
- R76 pad 2: VDD_EXT -> Net-(Q10-S)
- U17 pad 5: /SPI_ETH_INTERFACE_W5500/3V3A -> /SPI_ETH_INTERFACE_W5500/3V3D
- U26 pad P$10: Net-(Q12-C) -> /GSM_GPRS_MODULE_SIM7000G/MOSFET_LOGIC_LEVEL_TRANSLATOR/LOW_SIDE_LOGIC_SIGNAL
- U26 pad P$9: Net-(Q11-E) -> /GSM_GPRS_MODULE_SIM7000G/MOSFET_LOGIC_LEVEL_TRANSLATOR1/LOW_SIDE_LOGIC_SIGNAL
Routing:
- net /GSM_GPRS_MODULE_SIM7000G/MOSFET_LOGIC_LEVEL_TRANSLATOR/LOW_SIDE_LOGIC_SIGNAL: track 0.00 -> 12.3 mm
- net Net-(Q12-C): track 10.5 -> 0.00 mm
- net /GSM_GPRS_MODULE_SIM7000G/MOSFET_LOGIC_LEVEL_TRANSLATOR1/LOW_SIDE_LOGIC_SIGNAL: track 0.00 -> 8.42 mm
- net Net-(Q11-E): track 7.49 -> 0.00 mm
- net VDD_EXT: track 68.6 -> 74.0 mm, vias 4 -> 2
- net /SPI_ETH_INTERFACE_W5500/3V3A: track 67.4 -> 63.0 mm
- net Net-(J5-VBUS): track 8.00 -> 3.72 mm
- net /SPI_ETH_INTERFACE_W5500/3V3D: track 94.3 -> 98.4 mm
- net +24V: track 126.0 -> 122.4 mm
- net Net-(Q9-S): track 0.00 -> 3.16 mm
- net Net-(Q10-S): track 0.00 -> 3.10 mm
- net /ESP32_MCU/soft_uart_tx: track 54.3 -> 57.2 mm, vias 3 -> 5
- net /ESP32_MCU/~{esp_rst}: track 110.6 -> 108.1 mm
- net Net-(Q12-B): track 2.16 -> 0.00 mm
- net Net-(Q11-B): track 1.96 -> 0.00 mm
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- added copper zone on F.Cu, net Net-(C23-Pad1)
- added copper zone on B.Cu, net Net-(F1-Pad1)
Other:
- board text added: "3V3_EN"
