File: src/ELIESTER_V2/ELIESTER_V2.kicad_sch (KiCad schematic)
At the start: 12 parts, among them J1 Barrel_Jack_Switch, J2 SCREEN CONN FPC 10PIN 1MM, J6 Conn_01x04

Commit message: update on antenna an LAN side
Parts:
- J1: footprint Connector_BarrelJack:BarrelJack_GCT_DCJ200-10-A_Horizontal -> Connector_BarrelJack:BarrelJack_Horizontal
Changed lines of the file:
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@@
       (effects (font (size 1.27 1.27)))
     )
-    (property "Footprint" "Connector_BarrelJack:BarrelJack_GCT_DCJ200-10-A_Horizontal" (at 50.8 38.481 0)
+    (property "Footprint" "Connector_BarrelJack:BarrelJack_Horizontal" (at 50.8 38.481 0)
       (effects (font (size 1.27 1.27)) hide)
     )

Commit message: schematic update and gerber updates with corrections
Parts:
- added F1: JK30-250, greencharge-footprints:fuse-JK30-200, symbol Device:Polyfuse
- R1: value 2K -> 10R
Connections:
- net +24V: now also F1.2; no longer J1.1
- new net: F1.1, J1.1
Other:
- moved on the sheet: J6
